File: pcb/ecmd7/ecmd7.kicad_pcb (KiCad board)
At the start: 4 copper layers, 120 x 90 mm, 244 parts, among them J1 PMOD_SPI_ENC, J2 PMOD_ADC_MPIO, J3 PMOD_DRV, J4 Conn_01x02_Socket, J5 Encoder, J6 12V, J7 RS422/BISS-C, J8 5V, Q1 IRFS3806, Q10 BSC098N10NS5, Q11 MMBT3904, Q12 MMBT3904, Q2 IRFS3806, Q3 IRFS3806, Q4 IRFS3806, Q5 IRFS3806, Q6 IRFS3806, Q7 BSC098N10NS5, Q8 BSC098N10NS5, Q9 BSC098N10NS5, U1 TMC6200-TA, U10 FIN1002M5X, U11 FIN1002M5X, U12 FIN1002M5X, U13 ADM3490ExR, U14 LM5118MH, U15 74LVC1G139, U16 MB85RS1MT, U17 TMP122AIDBVR, U2 MCP33151-05T-E/MN, U3 LM5118MH, U4 MCP33151-05T-E/MN, U5 MCP33151-05T-E/MN, U6 TLV71318PDBV, U7 MCP33151-05T-E/MN, U9 LT1616ES6#TRPBF

Commit message: Final layout
Parts:
- removed D8: D, Diode_SMD:D_MiniMELF
- added D23: LL4148, Diode_SMD:D_MiniMELF, F.Cu at (83.0, 88.0)
- added H5: VMOT, MountingHole:MountingHole_3.2mm_M3_Pad_Via, F.Cu at (138.5, 45.0)
- added Logo: LOGO, LOGO, F.Cu at (102.2, 104.5)
- added R49: 330, Resistor_SMD:R_0805_2012Metric, F.Cu at (91.5, 100.5)
- added R53: 330, Resistor_SMD:R_0805_2012Metric, F.Cu at (86.3, 102.0)
- added R76: 330, Resistor_SMD:R_0805_2012Metric, F.Cu at (82.6, 102.0)
- added R9: 330, Resistor_SMD:R_0805_2012Metric, F.Cu at (89.5, 100.5)
- C23: value 4.7u -> 4.7u/25V
- C24: value 2.2u -> 2.2u/25V
- C37, C48: value 1u -> 1u/25V
- J6, J8: footprint Connector_PinHeader_2.54mm:PinHeader_1x02_P2.54mm_Vertical -> Connector_PinSocket_2.54mm:PinSocket_1x02_P2.54mm_Vertical
- JP1, JP5: value SolderJumper_2_Open -> 12V
- JP10: value SolderJumper_2_Bridged -> ~{WP}=1
- JP12: value SolderJumper_2_Open -> ~{WP}=0
- JP2, JP6: value SolderJumper_2_Bridged -> 5V
- JP3, JP9: value SolderJumper_2_Open -> INT
- JP4, JP7: value SolderJumper_2_Open -> 3V3
- JP8: value SolderJumper_2_Bridged -> EXT
- L3: value 10uH -> 10u
Routing:
- net +3.3V: track 318.6 -> 326.7 mm, vias 19 -> 21
- net SPI_SCK: track 114.6 -> 121.4 mm
- net SPI_SDO: track 147.3 -> 149.2 mm
- net /ADC+IO/~{CS_TMP}: track 44.2 -> 45.9 mm
- net GNDDRV: track 36.2 -> 34.8 mm, vias 57 -> 58
- net +5V: track 125.0 -> 126.0 mm, vias 9 -> 17
- net VMot: vias 82 -> 100
- net GNDMOT: vias 44 -> 117
- net GND: vias 168 -> 281
Other:
- board text added: "+"
- board text added: "-"
- board text added: "- -A+ - V B + +Z- +"
- board text added: "- 12V +"
- board text added: "- 5V +"
- board text added: "- B RX A V + B TX A"
- board text added: "12V"
- board text added: "3V3"
- board text added: "3V3(EN)"
- board text added: "5V"
- board text added: "BISS-C RS422 J7"
- board text added: "DRV"
- board text added: "ECMD7"
- board text added: "Encoder J5"
- board text added: "FAULT"
- board text added: "FRAM"
- board text added: "U"
- board text added: "V"
- board text added: "W"
- board text added: "©2025 S. Stähli"
